File: Hardware/PCBs/exp2/exp2.kicad_sch (KiCad schematic)
At the start: 8 parts, among them J1 Conn_01x11_Female, J2 Conn_01x06_Female, U1 74HC86, U2 7483

Commit message: Exp - 2 and 3 PCB Updated
Connections:
- net B0: now also U1.4; no longer U1.5
- net Cin: now also U1.5; no longer U1.4
Changed lines of the file:
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@@
 (kicad_sch (version 20211123) (generator eeschema)
   (paper "A4")
-  (junction (at 201.93 50.165) (diameter 0) (color 0 0 0 0)
-  )
   (junction (at 227.965 98.425) (diameter 0) (color 0 0 0 0)
   )
@@
   )
   (junction (at 153.67 50.165) (diameter 0) (color 0 0 0 0)
+  )
+  (junction (at 196.85 50.165) (diameter 0) (color 0 0 0 0)
   )
   (wire (pts (xy 122.555 70.485) (xy 122.555 68.58))
@@
     (stroke (width 0) (type default) (color 0 0 0 0))
   )
-  (wire (pts (xy 196.215 48.26) (xy 196.85 48.26))
+  (wire (pts (xy 196.215 48.26) (xy 201.93 48.26))
     (stroke (width 0) (type default) (color 0 0 0 0))
   )
@@
   )
   (wire (pts (xy 172.72 41.275) (xy 172.72 53.34))
-    (stroke (width 0) (type default) (color 0 0 0 0))
-  )
-  (wire (pts (xy 196.85 48.26) (xy 196.85 52.705))
     (stroke (width 0) (type default) (color 0 0 0 0))
   )
@@
     (stroke (width 0) (type default) (color 0 0 0 0))
   )
-  (wire (pts (xy 177.8 50.165) (xy 201.93 50.165))
+  (wire (pts (xy 177.8 50.165) (xy 196.85 50.165))
     (stroke (width 0) (type default) (color 0 0 0 0))
   )
@@
     (stroke (width 0) (type default) (color 0 0 0 0))
   )
-  (wire (pts (xy 201.93 50.165) (xy 201.93 52.705))
-    (stroke (width 0) (type default) (color 0 0 0 0))
-  )
   (wire (pts (xy 149.225 76.2) (xy 149.225 80.645))
     (stroke (width 0) (type default) (color 0 0 0 0))
@@
     (stroke (width 0) (type default) (color 0 0 0 0))
   )
-  (wire (pts (xy 201.93 50.165) (xy 238.125 50.165))
-    (stroke (width 0) (type default) (color 0 0 0 0))
-  )
   (wire (pts (xy 120.65 76.2) (xy 149.225 76.2))
     (stroke (width 0) (type default) (color 0 0 0 0))
@@
   )
   (wire (pts (xy 199.39 67.945) (xy 189.865 67.945))
+    (stroke (width 0) (type default) (color 0 0 0 0))
+  )
+  (wire (pts (xy 201.93 48.26) (xy 201.93 52.705))
     (stroke (width 0) (type default) (color 0 0 0 0))
   )
@@
     (stroke (width 0) (type default) (color 0 0 0 0))
   )
+  (wire (pts (xy 196.85 50.165) (xy 196.85 52.705))
+    (stroke (width 0) (type default) (color 0 0 0 0))
+  )
+  (wire (pts (xy 196.85 50.165) (xy 238.125 50.165))
+    (stroke (width 0) (type default) (color 0 0 0 0))
+  )
