File: Hardware/PCBs/exp11/exp11.kicad_sch (KiCad schematic)
At the start: 6 parts, among them J1 Conn_01x04_Female, J2 Conn_01x08_Female, U1 7432, U2 7408, U3 7404, U4 7495

Commit message: Multiple PCBs updated
Parts:
- added H1, H2, H3, H4: MountingHole, MountingHole:MountingHole_2.5mm, symbol Mechanical:MountingHole
Connections:
- net GND: no longer J2.7 (Pin_7), U1.14 (Vcc), U2.14 (Vcc), U2.14 (Vcc), U3.14 (Vcc), U3.14 (Vcc), U3.14 (Vcc), U4.14 (VCC)
- net QC: now reaches U2.1, U3.3, U4.11 (Q2)
- net QC: now also J2.2 (Pin_2); no longer J2.5 (Pin_5)
- net at U2.4: now also U3.6; no longer U3.5
- net CLK: now reaches U4.8 (~{CK2}), U4.9 (~{CK1})
- net CLK: now also J2.5 (Pin_5); no longer J2.1 (Pin_1)
- net MC: now reaches U4.6 (Mode)
- net MC: now also J2.6 (Pin_6); no longer J2.2 (Pin_2)
- net QA: now reaches J2.3 (Pin_3), U3.1, U4.13 (Q0)
- net QB: now reaches J2.4 (Pin_4), U4.12 (Q1)
- net A: now reaches J1.1 (Pin_1)
- net A: now also U4.2 (P0); no longer U4.5 (P3)
- net B: now reaches J1.2 (Pin_2)
- net B: now also U4.3 (P1); no longer U4.4 (P2)
- net C: now reaches J1.3 (Pin_3)
- net C: now also U4.4 (P2); no longer U4.3 (P1)
- net D: now reaches J1.4 (Pin_4)
- net D: now also U4.5 (P3); no longer U4.2 (P0)
- new net QD: J2.1 (Pin_1), U3.5, U4.10 (Q3)
- new net VCC: J2.7 (Pin_7), U1.14 (Vcc), U2.14 (Vcc), U2.14 (Vcc), U3.14 (Vcc), U3.14 (Vcc), U3.14 (Vcc), U4.14 (VCC)
Other:
- moved on the sheet: J1, J2, U3C
