File: Hardware/PCBs/exp11/exp11.kicad_pcb (KiCad board)
At the start: 2 copper layers, 55.9 x 38.1 mm, 10 parts, among them J1 Conn_01x04_Female, J2 Conn_01x08_Female, U1 7432, U2 7408, U3 7404, U4 7495

Commit message: PCBs Updated
Changed lines of the file:
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@@
     (fp_line (start 19 -0.7) (end -1.5 -0.7) (layer "F.Fab") (width 0.1))
     (fp_line (start -2.5 -6.7) (end 20 -6.7) (layer "F.Fab") (width 0.1))
-    (pad "1" thru_hole roundrect (at 0 0 90) (size 1.7 1.95) (drill 0.95) (layers *.Cu *.Mask) (roundrect_rratio 0.1470588235)
+    (pad "1" thru_hole roundrect (at 0 0 90) (size 1.7 1.95) (drill 1.2) (layers *.Cu *.Mask) (roundrect_rratio 0.1470588235)
       (net 10 "QD") (pinfunction "Pin_1") (pintype "passive"))
-    (pad "2" thru_hole oval (at 2.5 0 90) (size 1.7 1.95) (drill 0.95) (layers *.Cu *.Mask)
+    (pad "2" thru_hole oval (at 2.5 0 90) (size 1.7 1.95) (drill 1.2) (layers *.Cu *.Mask)
       (net 9 "QC") (pinfunction "Pin_2") (pintype "passive"))
-    (pad "3" thru_hole oval (at 5 0 90) (size 1.7 1.95) (drill 0.95) (layers *.Cu *.Mask)
+    (pad "3" thru_hole oval (at 5 0 90) (size 1.7 1.95) (drill 1.2) (layers *.Cu *.Mask)
       (net 7 "QA") (pinfunction "Pin_3") (pintype "passive"))
-    (pad "4" thru_hole oval (at 7.5 0 90) (size 1.7 1.95) (drill 0.95) (layers *.Cu *.Mask)
+    (pad "4" thru_hole oval (at 7.5 0 90) (size 1.7 1.95) (drill 1.2) (layers *.Cu *.Mask)
       (net 8 "QB") (pinfunction "Pin_4") (pintype "passive"))
-    (pad "5" thru_hole oval (at 10 0 90) (size 1.7 1.95) (drill 0.95) (layers *.Cu *.Mask)
+    (pad "5" thru_hole oval (at 10 0 90) (size 1.7 1.95) (drill 1.2) (layers *.Cu *.Mask)
       (net 5 "CLK") (pinfunction "Pin_5") (pintype "passive"))
-    (pad "6" thru_hole oval (at 12.5 0 90) (size 1.7 1.95) (drill 0.95) (layers *.Cu *.Mask)
+    (pad "6" thru_hole oval (at 12.5 0 90) (size 1.7 1.95) (drill 1.2) (layers *.Cu *.Mask)
       (net 6 "MC") (pinfunction "Pin_6") (pintype "passive"))
-    (pad "7" thru_hole oval (at 15 0 90) (size 1.7 1.95) (drill 0.95) (layers *.Cu *.Mask)
+    (pad "7" thru_hole oval (at 15 0 90) (size 1.7 1.95) (drill 1.2) (layers *.Cu *.Mask)
       (net 11 "VCC") (pinfunction "Pin_7") (pintype "passive"))
-    (pad "8" thru_hole oval (at 17.5 0 90) (size 1.7 1.95) (drill 0.95) (layers *.Cu *.Mask)
+    (pad "8" thru_hole oval (at 17.5 0 90) (size 1.7 1.95) (drill 1.2) (layers *.Cu *.Mask)
       (net 12 "GND") (pinfunction "Pin_8") (pintype "passive"))
     (model "${KICAD6_3DMODEL_DIR}/Connector_JST.3dshapes/JST_EH_S8B-EH_1x08_P2.50mm_Horizontal.wrl"
@@
     (fp_line (start -1.5 1.5) (end -2.5 1.5) (layer "F.Fab") (width 0.1))
     (fp_line (start -0.5 -0.7) (end 0 -1.407107) (layer "F.Fab") (width 0.1))
-    (pad "1" thru_hole roundrect (at 0 0 270) (size 1.7 1.95) (drill 0.95) (layers *.Cu *.Mask) (roundrect_rratio 0.1470588235)
+    (pad "1" thru_hole roundrect (at 0 0 270) (size 1.7 1.95) (drill 1.2) (layers *.Cu *.Mask) (roundrect_rratio 0.1470588235)
       (net 4 "A") (pinfunction "Pin_1") (pintype "passive"))
-    (pad "2" thru_hole oval (at 2.5 0 270) (size 1.7 1.95) (drill 0.95) (layers *.Cu *.Mask)
+    (pad "2" thru_hole oval (at 2.5 0 270) (size 1.7 1.95) (drill 1.2) (layers *.Cu *.Mask)
       (net 3 "B") (pinfunction "Pin_2") (pintype "passive"))
-    (pad "3" thru_hole oval (at 5 0 270) (size 1.7 1.95) (drill 0.95) (layers *.Cu *.Mask)
+    (pad "3" thru_hole oval (at 5 0 270) (size 1.7 1.95) (drill 1.2) (layers *.Cu *.Mask)
       (net 2 "C") (pinfunction "Pin_3") (pintype "passive"))
-    (pad "4" thru_hole oval (at 7.5 0 270) (size 1.7 1.95) (drill 0.95) (layers *.Cu *.Mask)
+    (pad "4" thru_hole oval (at 7.5 0 270) (size 1.7 1.95) (drill 1.2) (layers *.Cu *.Mask)
       (net 1 "D") (pinfunction "Pin_4") (pintype "passive"))
     (model "${KICAD6_3DMODEL_DIR}/Connector_JST.3dshapes/JST_EH_S4B-EH_1x04_P2.50mm_Horizontal.wrl"
