File: Hardware/PCBs/exp6a/exp6a.kicad_sch (KiCad schematic)
At the start: 5 parts, among them J1 Conn_01x04_Female, J2 Conn_01x03_Female, U1 7404, U2 7486, U3 7408

Commit message: updated exp 6a PCB
Parts:
- added H1, H2, H3, H4: MountingHole, MountingHole:MountingHole_2.5mm, symbol Mechanical:MountingHole
Connections:
- net Gnd: no longer J1.2 (Pin_2), U1.14 (Vcc), U1.14 (Vcc), U1.14 (Vcc), U2.14 (Vcc), U3.14 (Vcc), U3.14 (Vcc)
- net at J1.3 (Pin_3), U2.2, U3.5: now also U1.1; no longer U1.3
- net at U2.3: now also U1.13; no longer U1.1
- net at U3.2: now also U1.2; no longer U1.4
- net at J2.1 (Pin_1): now also U1.12; no longer U1.2
- new net Vcc: J1.2 (Pin_2), U1.14 (Vcc), U1.14 (Vcc), U1.14 (Vcc), U2.14 (Vcc), U3.14 (Vcc), U3.14 (Vcc)
Other:
- moved on the sheet: J1, J2, U1A, U1C, U1F, U2A, U3A, U3B

Commit message: Multiple PCBs updated
Connections:
- net A: now reaches J1.4 (Pin_4), U1.5, U2.1, U3.1
- net B: now reaches J1.3 (Pin_3), U1.1, U2.2, U3.5
- net Y3: now reaches J2.3 (Pin_3), U3.6
- net Y2: now reaches J2.1 (Pin_1), U1.12
- net Y1: now reaches J2.2 (Pin_2), U3.3
Changed lines of the file:
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@@
+    )
+  )
+  (global_label "A" (shape input) (at 91.44 66.04 90) (fields_autoplaced)
+    (effects (font (size 1.27 1.27)) (justify left))
+    (property "Intersheet References" "${INTERSHEET_REFS}" (id 0) (at 91.3606 62.5383 90)
+      (effects (font (size 1.27 1.27)) (justify left) hide)
     )
   )
@@
     )
   )
+  (global_label "Y3" (shape input) (at 210.82 114.3 0) (fields_autoplaced)
+    (effects (font (size 1.27 1.27)) (justify left))
+    (property "Intersheet References" "${INTERSHEET_REFS}" (id 0) (at 215.5312 114.2206 0)
+      (effects (font (size 1.27 1.27)) (justify left) hide)
+    )
+  )
   (global_label "VCC" (shape input) (at 149.86 63.5 90) (fields_autoplaced)
     (effects (font (size 1.27 1.27)) (justify left))
@@
     )
   )
+  (global_label "B" (shape input) (at 99.06 71.12 90) (fields_autoplaced)
+    (effects (font (size 1.27 1.27)) (justify left))
+    (property "Intersheet References" "${INTERSHEET_REFS}" (id 0) (at 98.9806 67.4369 90)
+      (effects (font (size 1.27 1.27)) (justify left) hide)
+    )
+  )
   (global_label "GND" (shape input) (at 109.22 85.09 180) (fields_autoplaced)
     (effects (font (size 1.27 1.27)) (justify right))
     (property "Intersheet References" "${INTERSHEET_REFS}" (id 0) (at 102.9364 85.1694 0)
       (effects (font (size 1.27 1.27)) (justify right) hide)
+    )
+  )
+  (global_label "Y2" (shape input) (at 209.55 68.58 0) (fields_autoplaced)
+    (effects (font (size 1.27 1.27)) (justify left))
+    (property "Intersheet References" "${INTERSHEET_REFS}" (id 0) (at 214.2612 68.5006 0)
+      (effects (font (size 1.27 1.27)) (justify left) hide)
     )
   )
@@
     )
   )
+  (global_label "Y1" (shape input) (at 203.2 83.82 90) (fields_autoplaced)
+    (effects (font (size 1.27 1.27)) (justify left))
+    (property "Intersheet References" "${INTERSHEET_REFS}" (id 0) (at 203.1206 79.1088 90)
+      (effects (font (size 1.27 1.27)) (justify left) hide)
+    )
+  )
