File: Hardware/PCBs/exp6a/exp6a.kicad_pcb (KiCad board)
At the start: 2 copper layers, 44.5 x 41.9 mm, 9 parts, among them J1 JST 4PIN F, J2 JST 3PIN F, U1 7404, U2 7486, U3 7408

Commit message: Multiple PCBs updated
Parts:
- J1: value JST 4PIN F -> A B Vcc Gnd
- J2: value JST 3PIN F -> Y3 Y1 Y2
Connections:
- net Net-(J1-Pad3) renamed B
- net Net-(J1-Pad4) renamed A
- net Net-(J2-Pad1) renamed Y2
- net Net-(J2-Pad2) renamed Y1
- net Net-(J2-Pad3) renamed Y3
Changed lines of the file:
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@@
   (net 1 "GND")
   (net 2 "VCC")
-  (net 3 "Net-(J1-Pad3)")
-  (net 4 "Net-(J1-Pad4)")
-  (net 5 "Net-(J2-Pad1)")
-  (net 6 "Net-(J2-Pad2)")
-  (net 7 "Net-(J2-Pad3)")
+  (net 3 "B")
+  (net 4 "A")
+  (net 5 "Y2")
+  (net 6 "Y1")
+  (net 7 "Y3")
   (net 8 "Net-(U1-Pad6)")
   (net 9 "Net-(U1-Pad2)")
@@
       (effects (font (size 1 1) (thickness 0.15)))
     )
-    (fp_text value "JST 4PIN F" (at 3.37 -5.4325 90) (layer "B.Cu")
+    (fp_text value "A B Vcc Gnd" (at 3.37 -5.4325 90) (layer "B.Cu")
       (effects (font (size 1 1) (thickness 0.25)) (justify mirror))
     )
@@
       (net 2 "VCC") (pinfunction "Pin_2") (pintype "passive"))
     (pad "3" thru_hole oval (at 5 0 90) (size 1.7 1.95) (drill 0.95) (layers *.Cu *.Mask)
-      (net 3 "Net-(J1-Pad3)") (pinfunction "Pin_3") (pintype "passive"))
+      (net 3 "B") (pinfunction "Pin_3") (pintype "passive"))
     (pad "4" thru_hole oval (at 7.5 0 90) (size 1.7 1.95) (drill 0.95) (layers *.Cu *.Mask)
-      (net 4 "Net-(J1-Pad4)") (pinfunction "Pin_4") (pintype "passive"))
+      (net 4 "A") (pinfunction "Pin_4") (pintype "passive"))
     (model "${KICAD6_3DMODEL_DIR}/Connector_JST.3dshapes/JST_EH_S4B-EH_1x04_P2.50mm_Horizontal.wrl"
       (offset (xyz 0 0 0))
@@
     (fp_line (start -1.27 16.57) (end 8.89 16.57) (layer "F.Fab") (width 0.1))
     (pad "1" thru_hole rect (at 0 0 90) (size 1.6 1.6) (drill 0.8) (layers *.Cu *.Mask)
-      (net 3 "Net-(J1-Pad3)") (pintype "input"))
+      (net 3 "B") (pintype "input"))
     (pad "2" thru_hole oval (at 0 2.54 90) (size 1.6 1.6) (drill 0.8) (layers *.Cu *.Mask)
       (net 9 "Net-(U1-Pad2)") (pintype "input"))
@@
     (pad "4" thru_hole oval (at 0 7.62 90) (size 1.6 1.6) (drill 0.8) (layers *.Cu *.Mask))
     (pad "5" thru_hole oval (at 0 10.16 90) (size 1.6 1.6) (drill 0.8) (layers *.Cu *.Mask)
-      (net 4 "Net-(J1-Pad4)") (pintype "input"))
+      (net 4 "A") (pintype "input"))
     (pad "6" thru_hole oval (at 0 12.7 90) (size 1.6 1.6) (drill 0.8) (layers *.Cu *.Mask)
       (net 8 "Net-(U1-Pad6)") (pintype "input"))
@@
     (pad "11" thru_hole oval (at 7.62 7.62 90) (size 1.6 1.6) (drill 0.8) (layers *.Cu *.Mask))
     (pad "12" thru_hole oval (at 7.62 5.08 90) (size 1.6 1.6) (drill 0.8) (layers *.Cu *.Mask)
-      (net 5 "Net-(J2-Pad1)") (pintype "input"))
+      (net 5 "Y2") (pintype "input"))
     (pad "13" thru_hole oval (at 7.62 2.54 90) (size 1.6 1.6) (drill 0.8) (layers *.Cu *.Mask)
       (net 10 "Net-(U1-Pad13)") (pintype "input"))
@@
     (fp_line (start 8.89 -1.33) (end -1.27 -1.33) (layer "F.Fab") (width 0.1))
     (pad "1" thru_hole rect (at 0 0 180) (size 1.6 1.6) (drill 0.8) (layers *.Cu *.Mask)
-      (net 4 "Net-(J1-Pad4)") (pintype "input"))
+      (net 4 "A") (pintype "input"))
     (pad "2" thru_hole oval (at 0 2.54 180) (size 1.6 1.6) (drill 0.8) (layers *.Cu *.Mask)
       (net 9 "Net-(U1-Pad2)") (pintype "input"))
     (pad "3" thru_hole oval (at 0 5.08 180) (size 1.6 1.6) (drill 0.8) (layers *.Cu *.Mask)
-      (net 6 "Net-(J2-Pad2)") (pintype "output"))
+      (net 6 "Y1") (pintype "output"))
     (pad "4" thru_hole oval (at 0 7.62 180) (size 1.6 1.6) (drill 0.8) (layers *.Cu *.Mask)
       (net 8 "Net-(U1-Pad6)") (pintype "input"))
     (pad "5" thru_hole oval (at 0 10.16 180) (size 1.6 1.6) (drill 0.8) (layers *.Cu *.Mask)
-      (net 3 "Net-(J1-Pad3)") (pintype "input"))
+      (net 3 "B") (pintype "input"))
     (pad "6" thru_hole oval (at 0 12.7 180) (size 1.6 1.6) (drill 0.8) (layers *.Cu *.Mask)
-      (net 7 "Net-(J2-Pad3)") (pintype "input"))
+      (net 7 "Y3") (pintype "input"))
     (pad "7" thru_hole oval (at 0 15.24 180) (size 1.6 1.6) (drill 0.8) (layers *.Cu *.Mask)
       (net 1 "GND") (pinfunction "Gnd") (pintype "power_in"))
@@
     (fp_line (start 6.985 -1.27) (end 6.985 16.51) (layer "F.Fab") (width 0.1))
     (pad "1" thru_hole rect (at 0 0 90) (size 1.6 1.6) (drill 0.8) (layers *.Cu *.Mask)
-      (net 4 "Net-(J1-Pad4)") (pintype "input"))
+      (net 4 "A") (pintype "input"))
     (pad "2" thru_hole oval (at 0 2.54 90) (size 1.6 1.6) (drill 0.8) (layers *.Cu *.Mask)
-      (net 3 "Net-(J1-Pad3)") (pintype "input"))
+      (net 3 "B") (pintype "input"))
     (pad "3" thru_hole oval (at 0 5.08 90) (size 1.6 1.6) (drill 0.8) (layers *.Cu *.Mask)
       (net 10 "Net-(U1-Pad13)") (pintype "output"))
@@
       (effects (font (size 1 1) (thickness 0.15)))
     )
-    (fp_text value "JST 3PIN F" (at 2.68 -5.5325 90) (layer "B.Cu")
+    (fp_text value "Y3 Y1 Y2" (at 2.5 -5.0725 270) (layer "B.Cu")
       (effects (font (size 1 1) (thickness 0.25)) (justify mirror))
     )
@@
     (fp_line (start -0.5 -0.7) (end 0 -1.407107) (layer "F.Fab") (width 0.1))
     (pad "1" thru_hole roundrect (at 0 0 90) (size 1.7 1.95) (drill 0.95) (layers *.Cu *.Mask) (roundrect_rratio 0.1470588235)
-      (net 5 "Net-(J2-Pad1)") (pinfunction "Pin_1") (pintype "passive"))
+      (net 5 "Y2") (pinfunction "Pin_1") (pintype "passive"))
     (pad "2" thru_hole oval (at 2.5 0 90) (size 1.7 1.95) (drill 0.95) (layers *.Cu *.Mask)
-      (net 6 "Net-(J2-Pad2)") (pinfunction "Pin_2") (pintype "passive"))
+      (net 6 "Y1") (pinfunction "Pin_2") (pintype "passive"))
     (pad "3" thru_hole oval (at 5 0 90) (size 1.7 1.95) (drill 0.95) (layers *.Cu *.Mask)
-      (net 7 "Net-(J2-Pad3)") (pinfunction "Pin_3") (pintype "passive"))
+      (net 7 "Y3") (pinfunction "Pin_3") (pintype "passive"))
     (model "${KICAD6_3DMODEL_DIR}/Connector_JST.3dshapes/JST_EH_S3B-EH_1x03_P2.50mm_Horizontal.wrl"
       (offset (xyz 0 0 0))
@@
     (effects (font (size 1.5 1.5) (thickness 0.3)) (justify mirror))
   )
+  (dimension (type aligned) (layer "Dwgs.User")
+    (pts (xy 119.38 76.2) (xy 163.83 76.2))
+    (height -3.81)
+    (gr_text "44.4500 mm" (at 141.605 71.24) (layer "Dwgs.User")
+      (effects (font (size 1 1) (thickness 0.15)))
+    )
+    (format (units 3) (units_format 1) (precision 4))
+    (style (thickness 0.15) (arrow_length 1.27) (text_position_mode 0) (extension_height 0.58642) (extension_offset 0.5) keep_text_aligned)
+  )
+  (dimension (type aligned) (layer "Dwgs.User")
+    (pts (xy 163.83 118.11) (xy 163.83 76.2))
+    (height 6.35)
+    (gr_text "41.9100 mm" (at 169.03 97.155 90) (layer "Dwgs.User")
+      (effects (font (size 1 1) (thickness 0.15)))
+    )
+    (format (units 3) (units_format 1) (precision 4))
+    (style (thickness 0.15) (arrow_length 1.27) (text_position_mode 0) (extension_height 0.58642) (extension_offset 0.5) keep_text_aligned)
+  )
   (segment (start 152.863604 107.46) (end 157.19 103.133604) (width 0.25) (layer "B.Cu") (net 1))

Commit message: PCBs Updated
Changed lines of the file:
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@@
     (fp_line (start -0.5 -0.7) (end 0 -1.407107) (layer "F.Fab") (width 0.1))
     (fp_line (start 10 -6.7) (end 10 1.5) (layer "F.Fab") (width 0.1))
-    (pad "1" thru_hole roundrect (at 0 0 90) (size 1.7 1.95) (drill 0.95) (layers *.Cu *.Mask) (roundrect_rratio 0.1470588235)
+    (pad "1" thru_hole roundrect (at 0 0 90) (size 1.7 1.95) (drill 1.2) (layers *.Cu *.Mask) (roundrect_rratio 0.1470588235)
       (net 1 "GND") (pinfunction "Pin_1") (pintype "passive"))
-    (pad "2" thru_hole oval (at 2.5 0 90) (size 1.7 1.95) (drill 0.95) (layers *.Cu *.Mask)
+    (pad "2" thru_hole oval (at 2.5 0 90) (size 1.7 1.95) (drill 1.2) (layers *.Cu *.Mask)
       (net 2 "VCC") (pinfunction "Pin_2") (pintype "passive"))
-    (pad "3" thru_hole oval (at 5 0 90) (size 1.7 1.95) (drill 0.95) (layers *.Cu *.Mask)
+    (pad "3" thru_hole oval (at 5 0 90) (size 1.7 1.95) (drill 1.2) (layers *.Cu *.Mask)
       (net 3 "B") (pinfunction "Pin_3") (pintype "passive"))
-    (pad "4" thru_hole oval (at 7.5 0 90) (size 1.7 1.95) (drill 0.95) (layers *.Cu *.Mask)
+    (pad "4" thru_hole oval (at 7.5 0 90) (size 1.7 1.95) (drill 1.2) (layers *.Cu *.Mask)
       (net 4 "A") (pinfunction "Pin_4") (pintype "passive"))
     (model "${KICAD6_3DMODEL_DIR}/Connector_JST.3dshapes/JST_EH_S4B-EH_1x04_P2.50mm_Horizontal.wrl"
@@
     (fp_line (start 7.5 1.5) (end 6.5 1.5) (layer "F.Fab") (width 0.1))
     (fp_line (start -0.5 -0.7) (end 0 -1.407107) (layer "F.Fab") (width 0.1))
-    (pad "1" thru_hole roundrect (at 0 0 90) (size 1.7 1.95) (drill 0.95) (layers *.Cu *.Mask) (roundrect_rratio 0.1470588235)
+    (pad "1" thru_hole roundrect (at 0 0 90) (size 1.7 1.95) (drill 1.2) (layers *.Cu *.Mask) (roundrect_rratio 0.1470588235)
       (net 5 "Y2") (pinfunction "Pin_1") (pintype "passive"))
-    (pad "2" thru_hole oval (at 2.5 0 90) (size 1.7 1.95) (drill 0.95) (layers *.Cu *.Mask)
+    (pad "2" thru_hole oval (at 2.5 0 90) (size 1.7 1.95) (drill 1.2) (layers *.Cu *.Mask)
       (net 6 "Y1") (pinfunction "Pin_2") (pintype "passive"))
-    (pad "3" thru_hole oval (at 5 0 90) (size 1.7 1.95) (drill 0.95) (layers *.Cu *.Mask)
+    (pad "3" thru_hole oval (at 5 0 90) (size 1.7 1.95) (drill 1.2) (layers *.Cu *.Mask)
       (net 7 "Y3") (pinfunction "Pin_3") (pintype "passive"))
     (model "${KICAD6_3DMODEL_DIR}/Connector_JST.3dshapes/JST_EH_S3B-EH_1x03_P2.50mm_Horizontal.wrl"
