File: Hardware/PCBs/exp6b/exp6b.kicad_sch (KiCad schematic)
At the start: 8 parts, among them J1 Conn_01x06_Female, J2 Conn_01x03_Female, U1 7404, U2 7408, U3 7486, U4 7408, U5 7404, U6 7432

Commit message: Multiple PCBs updated
Parts:
- added H1, H2, H3, H4: MountingHole, MountingHole:MountingHole_2.5mm, symbol Mechanical:MountingHole
- renumbered U5 to U1, U3 to U2, U4 to U3, U2 to U3, U6 to U4
Connections:
- net Gnd: now also J1.1 (Pin_1); no longer J1.5 (Pin_5), J1.6 (Pin_6), U1.14 (Vcc), U1.14 (Vcc), U1.14 (Vcc), U1.14 (Vcc), U1.14 (Vcc), U2.14 (Vcc), U2.14 (Vcc), U2.14 (Vcc), U2.14 (Vcc), U3.14 (Vcc), U3.14 (Vcc), U3.14 (Vcc), U3.14 (Vcc), U4.14 (Vcc)
- net at U4.1: now also U3.8; no longer U3.3
- net at U4.2: now also U3.6; no longer U3.6
- net Y1: now reaches U2.13, U4.3
- net Y1: now also J2.2 (Pin_2); no longer J2.3 (Pin_3)
- net at U2.8: now also U3.5; no longer U3.2
- net A1: now reaches U2.1, U2.10
- net A1: now also J1.4 (Pin_4), U3.9; no longer J1.1 (Pin_1), U3.5
- net B1: now reaches U1.1, U2.2
- net B1: now also J1.3 (Pin_3); no longer J1.4 (Pin_4)
- net at U2.3: now also U1.5; no longer U1.1
- net at U2.6: now also U1.9; no longer U1.3
- net at U2.11: now also U1.11; no longer U1.5
- net B0: now reaches U1.3, U2.5
- net B0: now also J1.2 (Pin_2); no longer J1.3 (Pin_3)
- net at U1.4: now also U3.2; no longer U3.1
- net at U1.2, U2.9: now also U3.10; no longer U3.4
- new net: U3.3, U3.4
- new net: U1.8, U3.13
- new net: U1.6, U3.12
- new net A0: J1.5 (Pin_5), U2.4, U3.1
- new net Vcc: J1.6 (Pin_6), U1.14 (Vcc), U1.14 (Vcc), U1.14 (Vcc), U1.14 (Vcc), U1.14 (Vcc), U2.14 (Vcc), U2.14 (Vcc), U2.14 (Vcc), U2.14 (Vcc), U3.14 (Vcc), U3.14 (Vcc), U3.14 (Vcc), U3.14 (Vcc), U4.14 (Vcc)
- new net Y2: J2.3 (Pin_3), U2.12, U3.11
- new net Y3: J2.1 (Pin_1), U1.10
Other:
- moved on the sheet: J1, J2, U1A, U1B, U1C, U1D, U1E, U2A, U2B, U2C, U2D, U3A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
